File: kicad/attiny-hvsp-programmer.kicad_pcb (KiCad board)
At the start: 2 copper layers, 13 parts, among them J1 Barrel_Jack, J3 Conn_02x04_Top_Bottom, Q1 2N3904, U1 ATtiny85-20P, U2 LM7805_TO220

Commit message: bugfix: add edge-cut
Other:
- board outline added: 40.6 x 45.7 mm
Changed lines of the file:
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@@
       (sketchpadsonfab false)
       (subtractmaskfromsilk false)
-      (outputformat 1)
+      (outputformat 5)
       (mirror false)
-      (drillshape 1)
+      (drillshape 0)
       (scaleselection 1)
-      (outputdirectory "")
+      (outputdirectory "./")
     )
   )
@@
       (effects (font (size 1 1) (thickness 0.15)))
     )
-    (fp_text value "LM7805_TO220" (at 2.54 2.5) (layer "F.Fab")
+    (fp_text value "LM7805_TO220" (at 2.54 7.691) (layer "F.Fab")
       (effects (font (size 1 1) (thickness 0.15)))
     )
@@
       (effects (font (size 1 1) (thickness 0.15)))
     )
-    (fp_text value "LED" (at 1.27 2.96 90) (layer "F.Fab")
+    (fp_text value "LED" (at 1.27 -5.08 90) (layer "F.Fab")
       (effects (font (size 1 1) (thickness 0.15)))
     )
@@
     )
   )
+  (gr_rect (start 139.7 83.82) (end 180.34 129.54) (layer "Edge.Cuts") (width 0.1) (fill none))
   (segment (start 165.1 104.14) (end 165.11 104.15) (width 0.25) (layer "F.Cu") (net 1))
   (segment (start 162.671 119.42) (end 162.56 119.309) (width 0.25) (layer "F.Cu") (net 1))
